File: T00R2/Design/T00R2.sch (EAGLE design)
At the start: 2 parts, among them P1 HEXABIT_17.32_TRIG_P1_P6

Commit message: -Update the Schematic logo -Extende the exposed copper space of the power pads at the angles -Improve the pins labling on the silkscreen
Other:
- note added: "T00R2"
- note added: "T00R2_Frontend"
- note removed: "0"
- note removed: "T00R20"
- note removed: "T00R20_Frontend"
